Commit message: #12: Edited Xacro and Driver Files

File: overlay_ws/src/KR240R2900_description/urdf/kr240r2900_2.xacro (robot description, xacro)
@@ -2,5 +2,19 @@
 <robot name="kr240r2900_2" xmlns:xacro="http://ros.org/wiki/xacro">
   <xacro:include filename="$(find kuka_robot_description)/urdf/kr240r2900_2_macro.xacro"/>
-  <xacro:kr240r2900_2 prefix=""/>
+  <xacro:arg name="controller_ip" default="0.0.0.0"/>
+  <xacro:arg name="client_ip" default="0.0.0.0"/>
+  <xacro:arg name="client_port" default="30200"/>
+  <xacro:arg name="use_fake_hardware" default="false"/>
+  <xacro:arg name="roundtrip_time" default="0"/>
+  <xacro:arg name="x" default="0"/>
+  <xacro:arg name="y" default="0"/>
+  <xacro:arg name="z" default="0"/>
+  <xacro:arg name="roll" default="0"/>
+  <xacro:arg name="pitch" default="0"/>
+  <xacro:arg name="yaw" default="0"/>
+  <xacro:arg name="prefix" default=""/>
+  <xacro:kr240r2900_2 prefix="$(arg prefix)" io_access="false" use_fake_hardware="$(arg use_fake_hardware)" roundtrip_time="$(arg roundtrip_time)" controller_ip="$(arg controller_ip)" client_ip="$(arg client_ip)" client_port="$(arg client_port)">
+      <origin xyz="$(arg x) $(arg y) $(arg z)" rpy="$(arg roll) $(arg pitch) $(arg yaw)"/>
+  </xacro:kr240r2900_2>
   <version>2024-11-08_16-30-13</version>
 </robot>
