Commit message: #16: Changes to URDF and Driver Launch Files

File: overlay_ws/src/kuka_kr240r2900_description/urdf/kr240r2900_2.xacro (robot description, xacro)
@@ -4,5 +4,5 @@
   <xacro:arg name="controller_ip" default="0.0.0.0"/>
   <xacro:arg name="client_ip" default="0.0.0.0"/>
-  <xacro:arg name="client_port" default="30200"/>
+  <xacro:arg name="client_port" default="59152"/>
   <xacro:arg name="use_fake_hardware" default="false"/>
   <xacro:arg name="roundtrip_time" default="0"/>
@@ -13,7 +13,6 @@
   <xacro:arg name="pitch" default="0"/>
   <xacro:arg name="yaw" default="0"/>
-  <xacro:arg name="prefix" default=""/>
-  <xacro:kr240r2900_2 prefix="$(arg prefix)" io_access="false" use_fake_hardware="$(arg use_fake_hardware)" roundtrip_time="$(arg roundtrip_time)" controller_ip="$(arg controller_ip)" client_ip="$(arg client_ip)" client_port="$(arg client_port)">
-      <origin xyz="$(arg x) $(arg y) $(arg z)" rpy="$(arg roll) $(arg pitch) $(arg yaw)"/>
+  <xacro:kr240r2900_2 client_ip="$(arg client_ip)" client_port="$(arg client_port)" prefix="$(arg prefix)" use_fake_hardware="$(arg use_fake_hardware)" roundtrip_time="$(arg roundtrip_time)">
+    <origin xyz="$(arg x) $(arg y) $(arg z)" rpy="$(arg roll) $(arg pitch) $(arg yaw)"/>
   </xacro:kr240r2900_2>
   <version>2024-11-08_16-30-13</version>

File: overlay_ws/src/kuka_kr240r2900_description/urdf/kr240r2900_2_macro.xacro (robot description, xacro)
@@ -1,4 +1,9 @@
 <?xml version='1.0' encoding='UTF-8'?>
 <robot xmlns:xacro="http://ros.org/wiki/xacro">
+  <xacro:include filename="$(find kuka_kr240r2900_description)/urdf/kr_quantec_ros2_control.xacro"/>
+  <xacro:include filename="$(find kuka_kr240r2900_description)/urdf/kr_quantec_transmission.xacro"/>
+  <xacro:macro name="kr240r2900_2" params="client_ip client_port prefix use_fake_hardware roundtrip_time *origin">
+  <!-- ros2 control instance -->
+  <xacro:kuka_quantec_ros2_control name="${prefix}kr240r2900_2" client_ip="${client_ip}" client_port="${client_port}" prefix="${prefix}" use_fake_hardware="${use_fake_hardware}" roundtrip_time="${roundtrip_time}"/>
   <xacro:property name="world" value="world"/>
   <xacro:property name="transmission_actuator_hw_interface" value="EffortJointInterface"/>
@@ -14,5 +19,5 @@
       <collision>
         <geometry>
-          <mesh filename="package://kuka_robot_description/meshes/kr240r2900_2/collision/base_link.stl"/>
+          <mesh filename="package://kuka_kr240r2900_description/meshes/kr240r2900_2/collision/base_link.stl"/>
         </geometry>
         <origin rpy="0.0 -0.0 0.0" xyz="0.0 0.0 0.0"/>
@@ -25,5 +30,5 @@
       <visual>
         <geometry>
-          <mesh filename="package://kuka_robot_description/meshes/kr240r2900_2/visual/base_link.dae"/>
+          <mesh filename="package://kuka_kr240r2900_description/meshes/kr240r2900_2/visual/base_link.dae"/>
         </geometry>
         <origin rpy="0.0 -0.0 0.0" xyz="0.0 0.0 0.0"/>
@@ -34,5 +39,5 @@
       <collision>
         <geometry>
-          <mesh filename="package://kuka_robot_description/meshes/kr240r2900_2/collision/link_1.stl"/>
+          <mesh filename="package://kuka_kr240r2900_description/meshes/kr240r2900_2/collision/link_1.stl"/>
         </geometry>
         <origin rpy="-3.141592653589793 0.0 -0.0" xyz="0.0 -3.742520618194312e-17 0.30560000000000004"/>
@@ -45,5 +50,5 @@
       <visual>
         <geometry>
-          <mesh filename="package://kuka_robot_description/meshes/kr240r2900_2/visual/link_1.dae"/>
+          <mesh filename="package://kuka_kr240r2900_description/meshes/kr240r2900_2/visual/link_1.dae"/>
         </geometry>
         <origin rpy="-3.141592653589793 0.0 -0.0" xyz="0.0 -3.742520618194312e-17 0.30560000000000004"/>
@@ -53,5 +58,5 @@
       <collision>
         <geometry>
-          <mesh filename="package://kuka_robot_description/meshes/kr240r2900_2/collision/link_2.stl"/>
+          <mesh filename="package://kuka_kr240r2900_description/meshes/kr240r2900_2/collision/link_2.stl"/>
         </geometry>
         <origin rpy="1.5707963267948968 -0.0 1.5707963267948966" xyz="-0.645 -0.32999999999999996 0.07200000000000009"/>
@@ -64,5 +69,5 @@
       <visual>
         <geometry>
-          <mesh filename="package://kuka_robot_description/meshes/kr240r2900_2/visual/link_2.dae"/>
+          <mesh filename="package://kuka_kr240r2900_description/meshes/kr240r2900_2/visual/link_2.dae"/>
         </geometry>
         <origin rpy="1.5707963267948968 -0.0 1.5707963267948966" xyz="-0.645 -0.32999999999999996 0.07200000000000009"/>
@@ -72,5 +77,5 @@
       <collision>
         <geometry>
-          <mesh filename="package://kuka_robot_description/meshes/kr240r2900_2/collision/link_3.stl"/>
+          <mesh filename="package://kuka_kr240r2900_description/meshes/kr240r2900_2/collision/link_3.stl"/>
         </geometry>
         <origin rpy="1.5707963267948968 -0.0 -0.0" xyz="-0.33000000000000007 1.995 0.1750000000000001"/>
@@ -83,5 +88,5 @@
       <visual>
         <geometry>
-          <mesh filename="package://kuka_robot_description/meshes/kr240r2900_2/visual/link_3.dae"/>
+          <mesh filename="package://kuka_kr240r2900_description/meshes/kr240r2900_2/visual/link_3.dae"/>
         </geometry>
         <origin rpy="1.5707963267948968 -0.0 -0.0" xyz="-0.33000000000000007 1.995 0.1750000000000001"/>
@@ -91,5 +96,5 @@
       <collision>
         <geometry>
-          <mesh filename="package://kuka_robot_description/meshes/kr240r2900_2/collision/link_4.stl"/>
+          <mesh filename="package://kuka_kr240r2900_description/meshes/kr240r2900_2/collision/link_4.stl"/>
         </geometry>
         <origin rpy="1.8369701987210297e-16 1.5707963267948966 0.0" xyz="-2.11 1.2451666974470345e-17 1.158"/>
@@ -102,5 +107,5 @@
       <visual>
         <geometry>
-          <mesh filename="package://kuka_robot_description/meshes/kr240r2900_2/visual/link_4.dae"/>
+          <mesh filename="package://kuka_kr240r2900_description/meshes/kr240r2900_2/visual/link_4.dae"/>
         </geometry>
         <origin rpy="1.8369701987210297e-16 1.5707963267948966 0.0" xyz="-2.11 1.2451666974470345e-17 1.158"/>
@@ -110,5 +115,5 @@
       <collision>
         <geometry>
-          <mesh filename="package://kuka_robot_description/meshes/kr240r2900_2/collision/link_5.stl"/>
+          <mesh filename="package://kuka_kr240r2900_description/meshes/kr240r2900_2/collision/link_5.stl"/>
         </geometry>
         <origin rpy="1.5707963267948968 -3.749399456654644e-33 -6.123233995736766e-17" xyz="-1.55 2.11 -0.1065"/>
@@ -121,5 +126,5 @@
       <visual>
         <geometry>
-          <mesh filename="package://kuka_robot_description/meshes/kr240r2900_2/visual/link_5.dae"/>
+          <mesh filename="package://kuka_kr240r2900_description/meshes/kr240r2900_2/visual/link_5.dae"/>
         </geometry>
         <origin rpy="1.5707963267948968 -3.749399456654644e-33 -6.123233995736766e-17" xyz="-1.55 2.11 -0.1065"/>
@@ -129,5 +134,5 @@
       <collision>
         <geometry>
-          <mesh filename="package://kuka_robot_description/meshes/kr240r2900_2/collision/link_6.stl"/>
+          <mesh filename="package://kuka_kr240r2900_description/meshes/kr240r2900_2/collision/link_6.stl"/>
         </geometry>
         <origin rpy="1.2246467991473532e-16 1.5707963267948966 0.0" xyz="-2.11 -1.233749536060084e-16 1.7194999999999998"/>
@@ -140,5 +145,5 @@
       <visual>
         <geometry>
-          <mesh filename="package://kuka_robot_description/meshes/kr240r2900_2/visual/link_6.dae"/>
+          <mesh filename="package://kuka_kr240r2900_description/meshes/kr240r2900_2/visual/link_6.dae"/>
         </geometry>
         <origin rpy="1.2246467991473532e-16 1.5707963267948966 0.0" xyz="-2.11 -1.233749536060084e-16 1.7194999999999998"/>
