Commit message: #17: Changed URDFs and Launch Files

File: overlay_ws/src/kr240r2900_2/urdf/kr240r2900_2_macro.xacro (robot description, xacro)
@@ -1,9 +1,4 @@
 <?xml version='1.0' encoding='UTF-8'?>
 <robot xmlns:xacro="http://ros.org/wiki/xacro">
-  <xacro:include filename="$(find kuka_kr240r2900_description)/urdf/kr_quantec_ros2_control.xacro"/>
-  <xacro:include filename="$(find kuka_kr240r2900_description)/urdf/kr_quantec_transmission.xacro"/>
-  <xacro:macro name="kr240r2900_2" params="client_ip client_port prefix use_fake_hardware roundtrip_time *origin">
-  <!-- ros2 control instance -->
-  <xacro:kuka_quantec_ros2_control name="${prefix}kr240r2900_2" client_ip="${client_ip}" client_port="${client_port}" prefix="${prefix}" use_fake_hardware="${use_fake_hardware}" roundtrip_time="${roundtrip_time}"/>
   <xacro:property name="world" value="world"/>
   <xacro:property name="transmission_actuator_hw_interface" value="EffortJointInterface"/>
@@ -19,5 +14,5 @@
       <collision>
         <geometry>
-          <mesh filename="package://kuka_kr240r2900_description/meshes/kr240r2900_2/collision/base_link.stl"/>
+          <mesh filename="package://kr240r2900_2/meshes/kr240r2900_2/collision/base_link.stl"/>
         </geometry>
         <origin rpy="0.0 -0.0 0.0" xyz="0.0 0.0 0.0"/>
@@ -30,5 +25,5 @@
       <visual>
         <geometry>
-          <mesh filename="package://kuka_kr240r2900_description/meshes/kr240r2900_2/visual/base_link.dae"/>
+          <mesh filename="package://kr240r2900_2/meshes/kr240r2900_2/visual/base_link.dae"/>
         </geometry>
         <origin rpy="0.0 -0.0 0.0" xyz="0.0 0.0 0.0"/>
@@ -39,5 +34,5 @@
       <collision>
         <geometry>
-          <mesh filename="package://kuka_kr240r2900_description/meshes/kr240r2900_2/collision/link_1.stl"/>
+          <mesh filename="package://kr240r2900_2/meshes/kr240r2900_2/collision/link_1.stl"/>
         </geometry>
         <origin rpy="-3.141592653589793 0.0 -0.0" xyz="0.0 -3.742520618194312e-17 0.30560000000000004"/>
@@ -50,5 +45,5 @@
       <visual>
         <geometry>
-          <mesh filename="package://kuka_kr240r2900_description/meshes/kr240r2900_2/visual/link_1.dae"/>
+          <mesh filename="package://kr240r2900_2/meshes/kr240r2900_2/visual/link_1.dae"/>
         </geometry>
         <origin rpy="-3.141592653589793 0.0 -0.0" xyz="0.0 -3.742520618194312e-17 0.30560000000000004"/>
@@ -58,5 +53,5 @@
       <collision>
         <geometry>
-          <mesh filename="package://kuka_kr240r2900_description/meshes/kr240r2900_2/collision/link_2.stl"/>
+          <mesh filename="package://kr240r2900_2/meshes/kr240r2900_2/collision/link_2.stl"/>
         </geometry>
         <origin rpy="1.5707963267948968 -0.0 1.5707963267948966" xyz="-0.645 -0.32999999999999996 0.07200000000000009"/>
@@ -69,5 +64,5 @@
       <visual>
         <geometry>
-          <mesh filename="package://kuka_kr240r2900_description/meshes/kr240r2900_2/visual/link_2.dae"/>
+          <mesh filename="package://kr240r2900_2/meshes/kr240r2900_2/visual/link_2.dae"/>
         </geometry>
         <origin rpy="1.5707963267948968 -0.0 1.5707963267948966" xyz="-0.645 -0.32999999999999996 0.07200000000000009"/>
@@ -77,5 +72,5 @@
       <collision>
         <geometry>
-          <mesh filename="package://kuka_kr240r2900_description/meshes/kr240r2900_2/collision/link_3.stl"/>
+          <mesh filename="package://kr240r2900_2/meshes/kr240r2900_2/collision/link_3.stl"/>
         </geometry>
         <origin rpy="1.5707963267948968 -0.0 -0.0" xyz="-0.33000000000000007 1.995 0.1750000000000001"/>
@@ -88,5 +83,5 @@
       <visual>
         <geometry>
-          <mesh filename="package://kuka_kr240r2900_description/meshes/kr240r2900_2/visual/link_3.dae"/>
+          <mesh filename="package://kr240r2900_2/meshes/kr240r2900_2/visual/link_3.dae"/>
         </geometry>
         <origin rpy="1.5707963267948968 -0.0 -0.0" xyz="-0.33000000000000007 1.995 0.1750000000000001"/>
@@ -96,5 +91,5 @@
       <collision>
         <geometry>
-          <mesh filename="package://kuka_kr240r2900_description/meshes/kr240r2900_2/collision/link_4.stl"/>
+          <mesh filename="package://kr240r2900_2/meshes/kr240r2900_2/collision/link_4.stl"/>
         </geometry>
         <origin rpy="1.8369701987210297e-16 1.5707963267948966 0.0" xyz="-2.11 1.2451666974470345e-17 1.158"/>
@@ -107,5 +102,5 @@
       <visual>
         <geometry>
-          <mesh filename="package://kuka_kr240r2900_description/meshes/kr240r2900_2/visual/link_4.dae"/>
+          <mesh filename="package://kr240r2900_2/meshes/kr240r2900_2/visual/link_4.dae"/>
         </geometry>
         <origin rpy="1.8369701987210297e-16 1.5707963267948966 0.0" xyz="-2.11 1.2451666974470345e-17 1.158"/>
@@ -115,5 +110,5 @@
       <collision>
         <geometry>
-          <mesh filename="package://kuka_kr240r2900_description/meshes/kr240r2900_2/collision/link_5.stl"/>
+          <mesh filename="package://kr240r2900_2/meshes/kr240r2900_2/collision/link_5.stl"/>
         </geometry>
         <origin rpy="1.5707963267948968 -3.749399456654644e-33 -6.123233995736766e-17" xyz="-1.55 2.11 -0.1065"/>
@@ -126,5 +121,5 @@
       <visual>
         <geometry>
-          <mesh filename="package://kuka_kr240r2900_description/meshes/kr240r2900_2/visual/link_5.dae"/>
+          <mesh filename="package://kr240r2900_2/meshes/kr240r2900_2/visual/link_5.dae"/>
         </geometry>
         <origin rpy="1.5707963267948968 -3.749399456654644e-33 -6.123233995736766e-17" xyz="-1.55 2.11 -0.1065"/>
@@ -134,5 +129,5 @@
       <collision>
         <geometry>
-          <mesh filename="package://kuka_kr240r2900_description/meshes/kr240r2900_2/collision/link_6.stl"/>
+          <mesh filename="package://kr240r2900_2/meshes/kr240r2900_2/collision/link_6.stl"/>
         </geometry>
         <origin rpy="1.2246467991473532e-16 1.5707963267948966 0.0" xyz="-2.11 -1.233749536060084e-16 1.7194999999999998"/>
@@ -145,5 +140,5 @@
       <visual>
         <geometry>
-          <mesh filename="package://kuka_kr240r2900_description/meshes/kr240r2900_2/visual/link_6.dae"/>
+          <mesh filename="package://kr240r2900_2/meshes/kr240r2900_2/visual/link_6.dae"/>
         </geometry>
         <origin rpy="1.2246467991473532e-16 1.5707963267948966 0.0" xyz="-2.11 -1.233749536060084e-16 1.7194999999999998"/>

File: overlay_ws/src/kuka_moveit_config/config/kr240r2900_2.urdf.xacro (robot description, xacro)
@@ -3,5 +3,5 @@
     <xacro:arg name="initial_positions_file" default="initial_positions.yaml" />
     <!-- Import kr240r2900_2 urdf file -->
-    <xacro:include filename="$(find kuka_robot_description)/urdf/kr240r2900_2.xacro" />
+    <xacro:include filename="$(find kr240r2900_2)/urdf/kr240r2900_2.xacro" />
     <!-- Import control_xacro -->
     <xacro:include filename="kr240r2900_2.ros2_control.xacro" />
