Commit message: #18: Updated URDFs and Driver Files

File: overlay_ws/src/kr240r2900_2/urdf/kr240r2900_2.xacro (robot description, xacro)
@@ -2,5 +2,20 @@
 <robot name="kr240r2900_2" xmlns:xacro="http://ros.org/wiki/xacro">
   <xacro:include filename="$(find kr240r2900_2)/urdf/kr240r2900_2_macro.xacro"/>
-  <xacro:kr240r2900_2 prefix=""/>
+  <!-- Read additional arguments  -->
+  <xacro:arg name="use_fake_hardware" default="true"/>
+  <xacro:arg name="mode" default="mock"/>
+  <xacro:arg name="roundtrip_time" default="0"/>
+  <xacro:arg name="client_ip" default="0.0.0.0"/>
+  <xacro:arg name="client_port" default="59152"/>
+  <xacro:arg name="prefix" default=""/>
+  <xacro:arg name="x" default="0"/>
+  <xacro:arg name="y" default="0"/>
+  <xacro:arg name="z" default="0"/>
+  <xacro:arg name="roll" default="0"/>
+  <xacro:arg name="pitch" default="0"/>
+  <xacro:arg name="yaw" default="0"/>
+  <xacro:kr240r2900_2 client_ip="$(arg client_ip)" client_port="$(arg client_port)" prefix="$(arg prefix)" use_fake_hardware="$(arg use_fake_hardware)" roundtrip_time="$(arg roundtrip_time)" mode="$(arg mode)">
+    <origin xyz="$(arg x) $(arg y) $(arg z)" rpy="$(arg roll) $(arg pitch) $(arg yaw)"/>
+  </xacro:kr240r2900_2>
   <version>2024-11-08_16-30-13</version>
 </robot>

File: overlay_ws/src/kr240r2900_2/urdf/kr240r2900_2_macro.xacro (robot description, xacro)
@@ -1,4 +1,6 @@
 <?xml version='1.0' encoding='UTF-8'?>
 <robot xmlns:xacro="http://ros.org/wiki/xacro">
+  <xacro:include filename="$(find kr240r2900_2)/urdf/kr_quantec_ros2_control.xacro"/>
+  <xacro:include filename="$(find kr240r2900_2)/urdf/kr_quantec_transmission.xacro"/>
   <xacro:property name="world" value="world"/>
   <xacro:property name="transmission_actuator_hw_interface" value="EffortJointInterface"/>
@@ -9,5 +11,7 @@
   <xacro:property name="base_joint_type" value="fixed"/>
   <xacro:property name="transmission_type" value="transmission_interface/SimpleTransmission"/>
-  <xacro:macro name="kr240r2900_2" params="prefix">
+  <xacro:macro name="kr240r2900_2" params="client_ip client_port prefix use_fake_hardware mode roundtrip_time *origin">
+    <!-- ros2 control instance -->
+    <xacro:kuka_quantec_ros2_control name="${prefix}kr240_r2900_2" client_ip="${client_ip}" client_port="${client_port}" prefix="${prefix}" use_fake_hardware="${use_fake_hardware}" roundtrip_time="${roundtrip_time}"/>
     <link name="${prefix}base"/>
     <link name="${prefix}base_link">

File: overlay_ws/src/kuka_moveit_config/config/kr240r2900_2.ros2_control.xacro (robot description, xacro)
@@ -10,61 +10,43 @@
             <joint name="joint_1">
                 <command_interface name="position"/>
-                <command_interface name="velocity"/>
-                <command_interface name="effort"/>
                 <state_interface name="position">
                   <param name="initial_value">${initial_positions['joint_1']}</param>
                 </state_interface>
                 <state_interface name="velocity"/>
-                <state_interface name="effort"/>
             </joint>
             <joint name="joint_2">
                 <command_interface name="position"/>
-                <command_interface name="velocity"/>
-                <command_interface name="effort"/>
                 <state_interface name="position">
                   <param name="initial_value">${initial_positions['joint_2']}</param>
                 </state_interface>
                 <state_interface name="velocity"/>
-                <state_interface name="effort"/>
             </joint>
             <joint name="joint_3">
                 <command_interface name="position"/>
-                <command_interface name="velocity"/>
-                <command_interface name="effort"/>
                 <state_interface name="position">
                   <param name="initial_value">${initial_positions['joint_3']}</param>
                 </state_interface>
                 <state_interface name="velocity"/>
-                <state_interface name="effort"/>
             </joint>
             <joint name="joint_4">
                 <command_interface name="position"/>
-                <command_interface name="velocity"/>
-                <command_interface name="effort"/>
                 <state_interface name="position">
                   <param name="initial_value">${initial_positions['joint_4']}</param>
                 </state_interface>
                 <state_interface name="velocity"/>
-                <state_interface name="effort"/>
             </joint>
             <joint name="joint_5">
                 <command_interface name="position"/>
-                <command_interface name="velocity"/>
-                <command_interface name="effort"/>
                 <state_interface name="position">
                   <param name="initial_value">${initial_positions['joint_5']}</param>
                 </state_interface>
                 <state_interface name="velocity"/>
-                <state_interface name="effort"/>
             </joint>
             <joint name="joint_6">
                 <command_interface name="position"/>
-                <command_interface name="velocity"/>
-                <command_interface name="effort"/>
                 <state_interface name="position">
                   <param name="initial_value">${initial_positions['joint_6']}</param>
                 </state_interface>
                 <state_interface name="velocity"/>
-                <state_interface name="effort"/>
             </joint>
         </ros2_control>

Commit message: #28: Removed Kuka Drivers

File: overlay_ws/src/kr240r2900_2/urdf/kr240r2900_2.xacro (robot description, xacro)
@@ -5,4 +5,5 @@
   <xacro:arg name="use_fake_hardware" default="true"/>
   <xacro:arg name="mode" default="mock"/>
+  <xacro:arg name="use_gpio" default="false"/>
   <xacro:arg name="roundtrip_time" default="0"/>
   <xacro:arg name="client_ip" default="0.0.0.0"/>

File: overlay_ws/src/kr240r2900_2/urdf/kr240r2900_2_macro.xacro (robot description, xacro)
@@ -11,7 +11,7 @@
   <xacro:property name="base_joint_type" value="fixed"/>
   <xacro:property name="transmission_type" value="transmission_interface/SimpleTransmission"/>
-  <xacro:macro name="kr240r2900_2" params="client_ip client_port prefix use_fake_hardware mode roundtrip_time *origin">
+  <xacro:macro name="kr240r2900_2" params="client_ip client_port prefix use_fake_hardware use_gpio mode roundtrip_time *origin">
     <!-- ros2 control instance -->
-    <xacro:kuka_quantec_ros2_control name="${prefix}kr240_r2900_2" client_ip="${client_ip}" client_port="${client_port}" prefix="${prefix}" use_fake_hardware="${use_fake_hardware}" roundtrip_time="${roundtrip_time}"/>
+    <xacro:kuka_quantec_ros2_control name="${prefix}kr240_r2900_2" client_ip="${client_ip}" client_port="${client_port}" prefix="${prefix}" use_fake_hardware="${use_fake_hardware}" roundtrip_time="${roundtrip_time}" use_gpio="$(use_gpio)"/>
     <link name="${prefix}base"/>
     <link name="${prefix}base_link">

File: overlay_ws/src/kr240r2900_2/urdf/kr_quantec_ros2_control.xacro (robot description, xacro)
@@ -53,4 +53,11 @@
         </state_interface>
       </joint>
+      <xacro:if value="${use_gpio}">
+        <xacro:include filename="$(find kuka_rsi_driver)/config/gpio_config.xacro"/>
+        <xacro:gpio_config/>
+      </xacro:if>
+      <xacro:unless value="${use_gpio}">
+        <gpio name="gpio"/>
+      </xacro:unless>
     </ros2_control>
   </xacro:macro>

Commit message: #29: Modified URDF Files

File: overlay_ws/src/kr240r2900_2/urdf/kr240r2900_2.xacro (robot description, xacro)
@@ -3,10 +3,12 @@
   <xacro:include filename="$(find kr240r2900_2)/urdf/kr240r2900_2_macro.xacro"/>
   <!-- Read additional arguments  -->
-  <xacro:arg name="use_fake_hardware" default="true"/>
-  <xacro:arg name="mode" default="mock"/>
+  <xacro:arg name="driver_version" default="rsi_only"/>
+  <xacro:arg name="use_fake_hardware" default="false"/>
+  <xacro:arg name="mode" default="hardware"/>
   <xacro:arg name="use_gpio" default="false"/>
   <xacro:arg name="roundtrip_time" default="0"/>
   <xacro:arg name="client_ip" default="0.0.0.0"/>
   <xacro:arg name="client_port" default="59152"/>
+  <xacro:arg name="controller_ip" default="0.0.0.0"/>
   <xacro:arg name="prefix" default=""/>
   <xacro:arg name="x" default="0"/>
@@ -16,5 +18,13 @@
   <xacro:arg name="pitch" default="0"/>
   <xacro:arg name="yaw" default="0"/>
-  <xacro:kr240r2900_2 client_ip="$(arg client_ip)" client_port="$(arg client_port)" prefix="$(arg prefix)" use_fake_hardware="$(arg use_fake_hardware)" roundtrip_time="$(arg roundtrip_time)" mode="$(arg mode)">
+  <xacro:kr240r2900_2 client_ip="$(arg client_ip)"
+                      client_port="$(arg client_port)"
+                      controller_ip="$(arg controller_ip)"
+                      prefix="$(arg prefix)"
+                      use_fake_hardware="$(arg use_fake_hardware)"
+                      roundtrip_time="$(arg roundtrip_time)"
+                      mode="$(arg mode)"
+                      use_gpio="$(arg use_gpio)"
+                      driver_version="$(arg driver_version)">
     <origin xyz="$(arg x) $(arg y) $(arg z)" rpy="$(arg roll) $(arg pitch) $(arg yaw)"/>
   </xacro:kr240r2900_2>

File: overlay_ws/src/kr240r2900_2/urdf/kr240r2900_2_macro.xacro (robot description, xacro)
@@ -11,7 +11,7 @@
   <xacro:property name="base_joint_type" value="fixed"/>
   <xacro:property name="transmission_type" value="transmission_interface/SimpleTransmission"/>
-  <xacro:macro name="kr240r2900_2" params="client_ip client_port prefix use_fake_hardware use_gpio mode roundtrip_time *origin">
+  <xacro:macro name="kr240r2900_2" params="client_ip client_port controller_ip prefix use_fake_hardware roundtrip_time use_gpio mode driver_version  *origin">
     <!-- ros2 control instance -->
-    <xacro:kuka_quantec_ros2_control name="${prefix}kr240_r2900_2" client_ip="${client_ip}" client_port="${client_port}" prefix="${prefix}" use_fake_hardware="${use_fake_hardware}" roundtrip_time="${roundtrip_time}" use_gpio="$(use_gpio)"/>
+    <xacro:kuka_quantec_ros2_control name="${prefix}kr240_r2900_2" client_ip="${client_ip}" client_port="${client_port}" prefix="${prefix}" use_fake_hardware="${use_fake_hardware}" roundtrip_time="${roundtrip_time}" use_gpio="${use_gpio}"/>
     <link name="${prefix}base"/>
     <link name="${prefix}base_link">

File: overlay_ws/src/kr240r2900_2/urdf/kr_quantec_ros2_control.xacro (robot description, xacro)
@@ -1,5 +1,5 @@
 <?xml version="1.0" encoding="UTF-8"?>
 <robot xmlns:xacro="http://www.ros.org/wiki/xacro">
-  <xacro:macro name="kuka_quantec_ros2_control" params="name client_ip client_port prefix use_fake_hardware roundtrip_time">
+  <xacro:macro name="kuka_quantec_ros2_control" params="name client_ip client_port prefix use_fake_hardware roundtrip_time use_gpio">
     <ros2_control name="${name}" type="system">
       <hardware>
@@ -12,5 +12,5 @@
         </xacro:if>
         <xacro:unless value="${use_fake_hardware}">
-          <plugin>kuka_kss_rsi_driver::KukaRSIHardwareInterface</plugin>
+          <plugin>kuka_rsi_driver::KukaRSIHardwareInterface</plugin>
           <param name="client_ip">${client_ip}</param>
           <param name="client_port">${client_port}</param>
