Commit message: #53: Modified omnimove.xacro  to include the LiDARs

File: overlay_ws/src/kr240_r2900_2/urdf/kr240_r2900_2.urdf.xacro (robot description, xacro)
@@ -14,7 +14,7 @@
   <xacro:arg name="verify_robot_model" default="true"/>
   <xacro:arg name="prefix" default=""/>
-  <xacro:arg name="x" default="0"/>
+  <xacro:arg name="x" default="0.9"/>   <!-- Changed from 0 -->
   <xacro:arg name="y" default="0"/>
-  <xacro:arg name="z" default="0"/>
+  <xacro:arg name="z" default="0.85"/>  <!-- Changed from 0 -->
   <xacro:arg name="roll" default="0"/>
   <xacro:arg name="pitch" default="0"/>

File: overlay_ws/src/kr240_r2900_2/urdf/omnimove_with_kr240_r2900_2.urdf.xacro (robot description, xacro)
@@ -3,11 +3,44 @@
   <xacro:include filename="$(find kr240_r2900_2)/urdf/kr240_r2900_2.urdf.xacro"/>
   <xacro:include filename="$(find kuka_omnimove_e575_support)/urdf/omnimove.xacro"/>
+  <xacro:include filename="$(find sick_safetyscanners2)/description/urdf/nanoscan3/nanoscan3_macro.xacro"/>
   <xacro:omnimove prefix="omnimove_"/>
   <xacro:omnimove_ros2_control name="omnimove"/>
-  <!-- attach the arm's 'world' to the omnimove base -->
+  <!-- place the omnimove on the world ground plane (omnimove_base is child of world)
+       Adjust the origin's z value if the mesh is not grounded at its link frame. -->
   <joint name="omni_to_world" type="fixed">
-    <parent link="omnimove_base"/>
-    <child link="world"/>
-    <origin xyz="0 1 0" rpy="0 0 0"/>
+    <parent link="world"/>
+    <child link="omnimove_base"/>
+    <origin xyz="0 0 0" rpy="0 0 0"/>
   </joint>
+  <!-- Add nanoscan3 sensors at specific locations on omnimove -->
+  <!-- Front-right sensor -->
+  <xacro:nanoscan3
+    name="nanoscan3_front_right"
+    parent="omnimove_platform"
+    mounting_kit="true"
+    ros_topic="/nanoscan3_front_right"
+    update_rate="50.0"
+    min_angle="${radians(-45)}"
+    max_angle="${radians(225)}"
+    min_range="0.05"
+    max_range="10.0"
+    gaussian_noise="0.006"
+    max_beams="500">
+    <origin xyz="1.55 -0.925 0.175" rpy="0 0 ${radians(-45)}" />
+  </xacro:nanoscan3>
+  <!-- Back-Left sensor -->
+  <xacro:nanoscan3
+    name="nanoscan3_front_left"
+    parent="omnimove_platform"
+    mounting_kit="true"
+    ros_topic="/nanoscan3_front_left"
+    update_rate="50.0"
+    min_angle="${radians(-45)}"
+    max_angle="${radians(225)}"
+    min_range="0.05"
+    max_range="10.0"
+    gaussian_noise="0.006"
+    max_beams="500">
+    <origin xyz="-1.55 0.925 0.175" rpy="0 0 ${radians(135)}" />
+  </xacro:nanoscan3>
 </robot>

File: overlay_ws/src/kuka_omnimove_e575_support/urdf/omnimove.xacro (robot description, xacro)
@@ -2,6 +2,43 @@
 <robot xmlns:xacro="http://wiki.ros.org/xacro" name="omnimove">
   <xacro:macro name="omnimove" params="prefix">
-    prefix="${prefix}"
       <link name="${prefix}base">
+        <inertial>
+          <mass value="0.01"/>
+          <inertia ixx="0.001" ixy="0.0" ixz="0.0" iyy="0.001" iyz="0.0" izz="0.001"/>
+        </inertial>
+      </link>
+      <!-- X axis prismatic joint -->
+      <joint name="${prefix}x_joint" type="prismatic">
+        <parent link="${prefix}base"/>
+        <child link="${prefix}x_link"/>
+        <axis xyz="1 0 0"/>
+        <limit lower="-10" upper="10" effort="1000" velocity="1.0"/>      </joint>
+      <link name="${prefix}x_link">
+        <inertial>
+          <mass value="0.01"/>
+          <inertia ixx="0.001" ixy="0.0" ixz="0.0" iyy="0.001" iyz="0.0" izz="0.001"/>
+        </inertial>
+      </link>
+      <!-- Y axis prismatic joint -->
+      <joint name="${prefix}y_joint" type="prismatic">
+        <parent link="${prefix}x_link"/>
+        <child link="${prefix}y_link"/>
+        <axis xyz="0 1 0"/>
+        <limit lower="-10" upper="10" effort="1000" velocity="1.0"/>
+      </joint>
+      <link name="${prefix}y_link">
+        <inertial>
+          <mass value="0.01"/>
+          <inertia ixx="0.001" ixy="0.0" ixz="0.0" iyy="0.001" iyz="0.0" izz="0.001"/>
+        </inertial>
+      </link>
+      <!-- Z axis rotational joint (rotation) -->
+      <joint name="${prefix}z_joint" type="revolute">
+        <parent link="${prefix}y_link"/>
+        <child link="${prefix}platform"/>
+        <axis xyz="0 0 1"/>
+        <limit lower="-3.14159" upper="3.14159" effort="1000" velocity="1.0"/>
+      </joint>
+      <link name="${prefix}platform">
         <visual>
           <origin xyz="0 0 0" rpy="0 0 0" />
@@ -21,5 +58,5 @@
 	    <ros2_control name="omnimove" type="system">
             <hardware>
-                <plugin>omnimove::KukaUTV3HardwareInterface</plugin>
+                <plugin>kuka_mock_hardware_interface::KukaMockHardwareInterface</plugin> <!-- Changed from omnimove::KukaUTV3HardwareInterface -->
                 <param name ="host">127.0.0.1</param>
                 <param name="port">24000</param>
