Commit message: #56: Integrated the Arm with omnimove

File: overlay_ws/src/kr240_r2900_2/urdf/kr240_r2900_2_macro.xacro (robot description, xacro)
@@ -195,9 +195,10 @@
       <parent link="${prefix}link_6"/>
     </joint>
-    <joint name="${prefix}world-base_link" type="fixed">
+    <!-- Commented out to allow the robot to be connected to the ominove platform instead of world -->
+    <!-- <joint name="${prefix}world-base_link" type="fixed">
       <child link="${prefix}base_link"/>
       <parent link="world"/>
       <xacro:insert_block name="origin"/>
-    </joint>
+    </joint> -->
   </xacro:macro>
 </robot>

File: overlay_ws/src/kr240_r2900_2/urdf/omnimove_with_kr240_r2900_2.urdf.xacro (robot description, xacro)
@@ -12,4 +12,9 @@
     <child link="omnimove_base"/>
     <origin xyz="0 0 0" rpy="0 0 0"/>
+  </joint>
+  <joint name="platform_to_arm_joint" type="fixed">
+    <parent link="omnimove_platform"/>
+    <child link="base_link"/>
+    <origin xyz="0.9 0 0.85" rpy="0 0 0"/>
   </joint>
   <!-- Add nanoscan3 sensors at specific locations on omnimove -->
@@ -31,8 +36,8 @@
   <!-- Back-Left sensor -->
   <xacro:nanoscan3
-    name="nanoscan3_front_left"
+    name="nanoscan3_back_left"
     parent="omnimove_platform"
     mounting_kit="true"
-    ros_topic="/nanoscan3_front_left"
+    ros_topic="/nanoscan3_back_left"
     update_rate="50.0"
     min_angle="${radians(-45)}"
