Commit message: #58: Fixed Moveit issue by creating dummy files

File: overlay_ws/src/kr240_r2900_2/urdf/kr240_r2900_2_macro_omni.xacro (robot description, xacro)
@@ -196,9 +196,9 @@
     </joint>
     <!-- Commented out to allow the robot to be connected to the ominove platform instead of world -->
-    <joint name="${prefix}world-base_link" type="fixed">
+    <!-- <joint name="${prefix}world-base_link" type="fixed">
       <child link="${prefix}base_link"/>
       <parent link="world"/>
       <xacro:insert_block name="origin"/>
-    </joint>
+    </joint> -->
   </xacro:macro>
 </robot>

File: overlay_ws/src/kr240_r2900_2/urdf/omnimove_with_kr240_r2900_2.urdf.xacro (robot description, xacro)
@@ -1,5 +1,5 @@
 <?xml version="1.0" ?>
 <robot name="kuka_with_omnimove" xmlns:xacro="http://wiki.ros.org/xacro">
-  <xacro:include filename="$(find kr240_r2900_2)/urdf/kr240_r2900_2.urdf.xacro"/>
+  <xacro:include filename="$(find kr240_r2900_2)/urdf/kr240_r2900_2_omni.urdf.xacro"/>
   <xacro:include filename="$(find kuka_omnimove_e575_support)/urdf/omnimove.xacro"/>
   <xacro:include filename="$(find sick_safetyscanners2)/description/urdf/nanoscan3/nanoscan3_macro.xacro"/>
